File: hardware/collar-reva/mcu.kicad_sch (KiCad schematic)
At the start: 7 parts, among them U1 ESP32-S3-MINI-1

Commit message: feat(collar): ESP32-S3 firmware and TI AFE4404 neck PPG
Host-tested HR/HRV, IMU RMS, and 1 Hz frames plus Arduino bring-up. Schematic adds the ventral-neck optical AFE on I2C so the puck can read pulse without actuation.

Co-authored-by: Cursor <cursoragent@cursor.com>
Other:
- note added: "SDA=GPIO4 SCL=GPIO5 I2S_SCK=GPIO7 I2S_WS=GPIO15 I2S_SD=GPIO16 IMU_INT=GPIO17 VBAT_SENSE=GPIO1 CHG_STAT=GPIO2 LED_STAT=GPIO6 PPG_RDY=GPIO8 PPG_RST=GPIO9"
- note removed: "SDA=GPIO4 SCL=GPIO5 I2S_SCK=GPIO7 I2S_WS=GPIO15 I2S_SD=GPIO16 IMU_INT=GPIO17 VBAT_SENSE=GPIO1 CHG_STAT=GPIO2 LED_STAT=GPIO6"
Changed lines of the file:
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@@
     (comment 2 "Observational wearable — no actuators on this board")
   )
-  (text "SDA=GPIO4  SCL=GPIO5  I2S_SCK=GPIO7  I2S_WS=GPIO15  I2S_SD=GPIO16  IMU_INT=GPIO17  VBAT_SENSE=GPIO1  CHG_STAT=GPIO2  LED_STAT=GPIO6" (at 20 18 0)
+  (text "SDA=GPIO4  SCL=GPIO5  I2S_SCK=GPIO7  I2S_WS=GPIO15  I2S_SD=GPIO16  IMU_INT=GPIO17  VBAT_SENSE=GPIO1  CHG_STAT=GPIO2  LED_STAT=GPIO6  PPG_RDY=GPIO8  PPG_RST=GPIO9" (at 20 18 0)
     (effects (font (size 1.27 1.27)) (justify left bottom))
   )
@@
     (effects (font (size 1.27 1.27)) (justify left))
   )
+  (global_label "PPG_RDY" (shape input) (at 155 120 0) (fields_autoplaced)
+    (effects (font (size 1.27 1.27)) (justify left))
+  )
+  (global_label "PPG_RST" (shape input) (at 155 125 0) (fields_autoplaced)
+    (effects (font (size 1.27 1.27)) (justify left))
+  )

Commit message: feat(hw): put photodiode, USB-C CC, and footprints on the Rev-A sheets
A C-to-C cable and neck PPG both need those parts on the schematic, not as layout notes. Footprints match the BOM so layout can start; copper is still the 30 mm outline.

Co-authored-by: Cursor <cursoragent@cursor.com>
Parts:
- C4: footprint (none) -> Capacitor_SMD:C_0402_1005Metric
- C5: footprint (none) -> Capacitor_SMD:C_0805_2012Metric
- D2: footprint (none) -> LED_SMD:LED_0402_1005Metric
- R4, R5, R6: footprint (none) -> Resistor_SMD:R_0402_1005Metric
- U1: footprint (none) -> RF_Module:ESP32-S3-MINI-1
Changed lines of the file:
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@@
       (effects (font (size 1.27 1.27)))
     )
-    (property "Footprint" "" (at 110 80 0)
+    (property "Footprint" "RF_Module:ESP32-S3-MINI-1" (at 110 80 0)
       (effects (font (size 1.27 1.27)) hide)
     )
@@
       (effects (font (size 1.27 1.27)))
     )
-    (property "Footprint" "" (at 70 55 0)
+    (property "Footprint" "Resistor_SMD:R_0402_1005Metric" (at 70 55 0)
       (effects (font (size 1.27 1.27)) hide)
     )
@@
       (effects (font (size 1.27 1.27)))
     )
-    (property "Footprint" "" (at 70 80 0)
+    (property "Footprint" "Resistor_SMD:R_0402_1005Metric" (at 70 80 0)
       (effects (font (size 1.27 1.27)) hide)
     )
@@
       (effects (font (size 1.27 1.27)))
     )
-    (property "Footprint" "" (at 160 110 0)
+    (property "Footprint" "Resistor_SMD:R_0402_1005Metric" (at 160 110 0)
       (effects (font (size 1.27 1.27)) hide)
     )
@@
       (effects (font (size 1.27 1.27)))
     )
-    (property "Footprint" "" (at 175 110 0)
+    (property "Footprint" "LED_SMD:LED_0402_1005Metric" (at 175 110 0)
       (effects (font (size 1.27 1.27)) hide)
     )
@@
       (effects (font (size 1.27 1.27)))
     )
-    (property "Footprint" "" (at 80 45 0)
+    (property "Footprint" "Capacitor_SMD:C_0402_1005Metric" (at 80 45 0)
       (effects (font (size 1.27 1.27)) hide)
     )
@@
       (effects (font (size 1.27 1.27)))
     )
-    (property "Footprint" "" (at 95 45 0)
+    (property "Footprint" "Capacitor_SMD:C_0805_2012Metric" (at 95 45 0)
       (effects (font (size 1.27 1.27)) hide)
     )

Commit message: feat(collar): emit gyro, die temp, and neck NTC on the 1 Hz map
The BMI270 and AFE already had unused channels. Turn them on and stuff the missing red LED plus contact NTC so the same notify map can carry chemistry-adjacent proxies without a new protocol.

Co-authored-by: Cursor <cursoragent@cursor.com>
Other:
- note added: "SDA=GPIO4 SCL=GPIO5 I2S_SCK=GPIO7 I2S_WS=GPIO15 I2S_SD=GPIO16 IMU_INT=GPIO17 VBAT_SENSE=GPIO1 CHG_STAT=GPIO2 LED_STAT=GPIO6 PPG_RDY=GPIO8 PPG_RST=GPIO9 SKIN_SENSE=GPIO10"
- note removed: "SDA=GPIO4 SCL=GPIO5 I2S_SCK=GPIO7 I2S_WS=GPIO15 I2S_SD=GPIO16 IMU_INT=GPIO17 VBAT_SENSE=GPIO1 CHG_STAT=GPIO2 LED_STAT=GPIO6 PPG_RDY=GPIO8 PPG_RST=GPIO9"
Changed lines of the file:
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@@
     (comment 2 "Observational wearable — no actuators on this board")
   )
-  (text "SDA=GPIO4  SCL=GPIO5  I2S_SCK=GPIO7  I2S_WS=GPIO15  I2S_SD=GPIO16  IMU_INT=GPIO17  VBAT_SENSE=GPIO1  CHG_STAT=GPIO2  LED_STAT=GPIO6  PPG_RDY=GPIO8  PPG_RST=GPIO9" (at 20 18 0)
+  (text "SDA=GPIO4  SCL=GPIO5  I2S_SCK=GPIO7  I2S_WS=GPIO15  I2S_SD=GPIO16  IMU_INT=GPIO17  VBAT_SENSE=GPIO1  CHG_STAT=GPIO2  LED_STAT=GPIO6  PPG_RDY=GPIO8  PPG_RST=GPIO9  SKIN_SENSE=GPIO10" (at 20 18 0)
     (effects (font (size 1.27 1.27)) (justify left bottom))
   )
@@
     (pin "13")
     (pin "14")
+    (pin "15")
     (instances
       (project "collar-reva"
@@
     (effects (font (size 1.27 1.27)) (justify left))
   )
+  (global_label "SKIN_SENSE" (shape input) (at 85 115 0) (fields_autoplaced)
+    (effects (font (size 1.27 1.27)) (justify left))
+  )
