File: hardware/collar-reva/mcu.kicad_sch (KiCad schematic)
At the start: 7 parts, among them U1 ESP32-S3-MINI-1

Commit message: feat(collar): ESP32-S3 firmware and neck PPG (#34)
* feat(collar): ESP32-S3 firmware and TI AFE4404 neck PPG

Host-tested HR/HRV, IMU RMS, and 1 Hz frames plus Arduino bring-up. Schematic adds the ventral-neck optical AFE on I2C so the puck can read pulse without actuation.

Co-authored-by: Cursor <cursoragent@cursor.com>

* feat(firmware): wire IMU, VBAT, and audio features into the collar loop

Bring-up now reads BMI270 accel and AFE4404 IR, converts VBAT on the derived divider, and keeps BLE notify-only.

Co-authored-by: Cursor <cursoragent@cursor.com>

* feat(firmware): I2S mic hop and VBAT-empty fault priority

INMP441 now feeds audio RMS/bark on the Rev-A pin map, and a low cell overrides a missing PPG peak so the 1 Hz frame reports the more urgent fault.

Co-authored-by: Cursor <cursoragent@cursor.com>

* feat(firmware): emit Phase-2 CBOR frames and check BMI270 chip ID

The 1 Hz notify is a real CBOR map (not JSON), and bring-up NAKs a missing IMU so we do not silently stream zeros.

Co-authored-by: Cursor <cursoragent@cursor.com>

* docs(firmware): note I2S RX pins in the collar bring-up order

Co-authored-by: Cursor <cursoragent@cursor.com>

* feat(firmware): pack 1 Hz CBOR to a BLE notify MTU

Frames now clip to MTU-3 so a default 23-byte ATT MTU cannot silently truncate the Phase-2 map once NimBLE is attached.

Co-authored-by: Cursor <cursoragent@cursor.com>

* feat(firmware): NimBLE advertise aarf-collar and notify 1 Hz CBOR

Phone can subscribe to the notify-only GATT char. LED and WDT follow the fault table, and IMU/mic NAKs now beat a missing PPG peak.

Co-authored-by: Cursor <cursoragent@cursor.com>

* feat(firmware): BMI270 accel bring-up and NVS VBAT cal

Soft-reset and enable ±8 g accel after chip-ID, and load divider scale/offset from NVS so bench cal survives reboot. PlatformIO build stays green.

Co-authored-by: Cursor <cursoragent@cursor.com>

* feat(firmware): bark CLIP to /infer/audio plus AFE4404 4 mA init

Wi-Fi posts the existing runtime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
Parts:
- C4: footprint (none) -> Capacitor_SMD:C_0402_1005Metric
- C5: footprint (none) -> Capacitor_SMD:C_0805_2012Metric
- D2: footprint (none) -> LED_SMD:LED_0402_1005Metric
- R4, R5, R6: footprint (none) -> Resistor_SMD:R_0402_1005Metric
- U1: footprint (none) -> RF_Module:ESP32-S3-MINI-1
Other:
- note added: "SDA=GPIO4 SCL=GPIO5 I2S_SCK=GPIO7 I2S_WS=GPIO15 I2S_SD=GPIO16 IMU_INT=GPIO17 VBAT_SENSE=GPIO1 CHG_STAT=GPIO2 LED_STAT=GPIO6 PPG_RDY=GPIO8 PPG_RST=GPIO9 SKIN_SENSE=GPIO10"
- note removed: "SDA=GPIO4 SCL=GPIO5 I2S_SCK=GPIO7 I2S_WS=GPIO15 I2S_SD=GPIO16 IMU_INT=GPIO17 VBAT_SENSE=GPIO1 CHG_STAT=GPIO2 LED_STAT=GPIO6"
Changed lines of the file:
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@@
     (comment 2 "Observational wearable — no actuators on this board")
   )
-  (text "SDA=GPIO4  SCL=GPIO5  I2S_SCK=GPIO7  I2S_WS=GPIO15  I2S_SD=GPIO16  IMU_INT=GPIO17  VBAT_SENSE=GPIO1  CHG_STAT=GPIO2  LED_STAT=GPIO6" (at 20 18 0)
+  (text "SDA=GPIO4  SCL=GPIO5  I2S_SCK=GPIO7  I2S_WS=GPIO15  I2S_SD=GPIO16  IMU_INT=GPIO17  VBAT_SENSE=GPIO1  CHG_STAT=GPIO2  LED_STAT=GPIO6  PPG_RDY=GPIO8  PPG_RST=GPIO9  SKIN_SENSE=GPIO10" (at 20 18 0)
     (effects (font (size 1.27 1.27)) (justify left bottom))
   )
@@
       (effects (font (size 1.27 1.27)))
     )
-    (property "Footprint" "" (at 110 80 0)
+    (property "Footprint" "RF_Module:ESP32-S3-MINI-1" (at 110 80 0)
       (effects (font (size 1.27 1.27)) hide)
     )
@@
     (pin "13")
     (pin "14")
+    (pin "15")
     (instances
       (project "collar-reva"
@@
       (effects (font (size 1.27 1.27)))
     )
-    (property "Footprint" "" (at 70 55 0)
+    (property "Footprint" "Resistor_SMD:R_0402_1005Metric" (at 70 55 0)
       (effects (font (size 1.27 1.27)) hide)
     )
@@
       (effects (font (size 1.27 1.27)))
     )
-    (property "Footprint" "" (at 70 80 0)
+    (property "Footprint" "Resistor_SMD:R_0402_1005Metric" (at 70 80 0)
       (effects (font (size 1.27 1.27)) hide)
     )
@@
       (effects (font (size 1.27 1.27)))
     )
-    (property "Footprint" "" (at 160 110 0)
+    (property "Footprint" "Resistor_SMD:R_0402_1005Metric" (at 160 110 0)
       (effects (font (size 1.27 1.27)) hide)
     )
@@
       (effects (font (size 1.27 1.27)))
     )
-    (property "Footprint" "" (at 175 110 0)
+    (property "Footprint" "LED_SMD:LED_0402_1005Metric" (at 175 110 0)
       (effects (font (size 1.27 1.27)) hide)
     )
@@
       (effects (font (size 1.27 1.27)))
     )
-    (property "Footprint" "" (at 80 45 0)
+    (property "Footprint" "Capacitor_SMD:C_0402_1005Metric" (at 80 45 0)
       (effects (font (size 1.27 1.27)) hide)
     )
@@
       (effects (font (size 1.27 1.27)))
     )
-    (property "Footprint" "" (at 95 45 0)
+    (property "Footprint" "Capacitor_SMD:C_0805_2012Metric" (at 95 45 0)
       (effects (font (size 1.27 1.27)) hide)
     )
@@
     (effects (font (size 1.27 1.27)) (justify left))
   )
+  (global_label "PPG_RDY" (shape input) (at 155 120 0) (fields_autoplaced)
+    (effects (font (size 1.27 1.27)) (justify left))
+  )
+  (global_label "PPG_RST" (shape input) (at 155 125 0) (fields_autoplaced)
+    (effects (font (size 1.27 1.27)) (justify left))
+  )
+  (global_label "SKIN_SENSE" (shape input) (at 85 115 0) (fields_autoplaced)
+    (effects (font (size 1.27 1.27)) (justify left))
+  )
