File: hardware/collar-reva/sensors.kicad_sch (KiCad schematic)
At the start: 6 parts, among them U4 BMI270, U5 INMP441

Commit message: feat(collar): ESP32-S3 firmware and neck PPG (#34)
* feat(collar): ESP32-S3 firmware and TI AFE4404 neck PPG

Host-tested HR/HRV, IMU RMS, and 1 Hz frames plus Arduino bring-up. Schematic adds the ventral-neck optical AFE on I2C so the puck can read pulse without actuation.

Co-authored-by: Cursor <cursoragent@cursor.com>

* feat(firmware): wire IMU, VBAT, and audio features into the collar loop

Bring-up now reads BMI270 accel and AFE4404 IR, converts VBAT on the derived divider, and keeps BLE notify-only.

Co-authored-by: Cursor <cursoragent@cursor.com>

* feat(firmware): I2S mic hop and VBAT-empty fault priority

INMP441 now feeds audio RMS/bark on the Rev-A pin map, and a low cell overrides a missing PPG peak so the 1 Hz frame reports the more urgent fault.

Co-authored-by: Cursor <cursoragent@cursor.com>

* feat(firmware): emit Phase-2 CBOR frames and check BMI270 chip ID

The 1 Hz notify is a real CBOR map (not JSON), and bring-up NAKs a missing IMU so we do not silently stream zeros.

Co-authored-by: Cursor <cursoragent@cursor.com>

* docs(firmware): note I2S RX pins in the collar bring-up order

Co-authored-by: Cursor <cursoragent@cursor.com>

* feat(firmware): pack 1 Hz CBOR to a BLE notify MTU

Frames now clip to MTU-3 so a default 23-byte ATT MTU cannot silently truncate the Phase-2 map once NimBLE is attached.

Co-authored-by: Cursor <cursoragent@cursor.com>

* feat(firmware): NimBLE advertise aarf-collar and notify 1 Hz CBOR

Phone can subscribe to the notify-only GATT char. LED and WDT follow the fault table, and IMU/mic NAKs now beat a missing PPG peak.

Co-authored-by: Cursor <cursoragent@cursor.com>

* feat(firmware): BMI270 accel bring-up and NVS VBAT cal

Soft-reset and enable ±8 g accel after chip-ID, and load divider scale/offset from NVS so bench cal survives reboot. PlatformIO build stays green.

Co-authored-by: Cursor <cursoragent@cursor.com>

* feat(firmware): bark CLIP to /infer/audio plus AFE4404 4 mA init

Wi-Fi posts the existing runtime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
Parts:
- added C8: 0.1uF PPG, Capacitor_SMD:C_0402_1005Metric, symbol Device:C
- added D3: IR neck, LED_SMD:LED_0805_2012Metric, symbol Device:LED
- added D4: PD neck, Diode_SMD:D_0805_2012Metric, symbol Device:LED
- added D5: RED neck, LED_SMD:LED_0805_2012Metric, symbol Device:LED
- added R11, RT1: 10k NTC, Resistor_SMD:R_0402_1005Metric, symbol Device:R
- added U6: AFE4404, Package_BGA:Texas_DSBGA-15_1.91x1.91mm_Layout5x3_P0.4mm, symbol aarf:PPG
- C6, C7: footprint (none) -> Capacitor_SMD:C_0402_1005Metric
- R7, R8: footprint (none) -> Resistor_SMD:R_0402_1005Metric
- U4: footprint (none) -> Sensor_Motion:Bosch_LGA-14_2.5x3mm_P0.5mm_ClockwisePinNumbering
- U5: footprint (none) -> Sensor_Audio:InvenSense_INMP441
Other:
- note added: "D5 is 660 nm on AFE LED2. RT1 is neck-contact NTC, not core temp. Not SpO2."
- note added: "I2C pull-ups 4.7k. AFE4404 optical AFE faces the ventral neck (carotid)."
- note removed: "I2C pull-ups 4.7k to 3V3. INMP441 L/R tied to GND (left channel)."
Changed lines of the file:
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@@
     (date "2026-08-21")
     (rev "A")
-    (comment 1 "BMI270 I2C + INMP441 I2S. Clean analog/digital island.")
+    (comment 1 "BMI270 + INMP441 + TI AFE4404 neck PPG.")
     (comment 2 "Observational wearable — no actuators on this board")
   )
-  (text "I2C pull-ups 4.7k to 3V3. INMP441 L/R tied to GND (left channel)." (at 20 20 0)
+  (text "I2C pull-ups 4.7k. AFE4404 optical AFE faces the ventral neck (carotid)." (at 20 20 0)
     (effects (font (size 1.27 1.27)) (justify left bottom))
   )
+  (text "D5 is 660 nm on AFE LED2. RT1 is neck-contact NTC, not core temp. Not SpO2." (at 20 24 0)
+    (effects (font (size 1.27 1.27)) (justify left bottom))
+  )
   (symbol (lib_id "aarf:IMU") (at 80 70 0) (unit 1)
     (in_bom yes) (on_board yes)
@@
       (effects (font (size 1.27 1.27)))
     )
-    (property "Footprint" "" (at 80 70 0)
+    (property "Footprint" "Sensor_Motion:Bosch_LGA-14_2.5x3mm_P0.5mm_ClockwisePinNumbering" (at 80 70 0)
       (effects (font (size 1.27 1.27)) hide)
     )
@@
       (effects (font (size 1.27 1.27)))
     )
-    (property "Footprint" "" (at 160 70 0)
+    (property "Footprint" "Sensor_Audio:InvenSense_INMP441" (at 160 70 0)
       (effects (font (size 1.27 1.27)) hide)
     )
@@
     )
   )
+  (symbol (lib_id "aarf:PPG") (at 80 140 0) (unit 1)
+    (in_bom yes) (on_board yes)
+    (property "Reference" "U6" (at 80 127.3 0)
+      (effects (font (size 1.27 1.27)))
+    )
+    (property "Value" "AFE4404" (at 80 152.7 0)
+      (effects (font (size 1.27 1.27)))
+    )
+    (property "Footprint" "Package_BGA:Texas_DSBGA-15_1.91x1.91mm_Layout5x3_P0.4mm" (at 80 140 0)
+      (effects (font (size 1.27 1.27)) hide)
+    )
+    (property "Datasheet" "~" (at 80 140 0)
+      (effects (font (size 1.27 1.27)) hide)
+    )
+    (pin "1")
+    (pin "2")
+    (pin "3")
+    (pin "4")
+    (pin "5")
+    (pin "6")
+    (pin "7")
+    (pin "8")
+    (pin "9")
+    (instances
+      (project "collar-reva"
+        (path "/7fffe17a-9ffb-4f1f-b4b6-a4342b258eee/72e61ef2-c28b-4186-b83a-fe973384e252"
+          (reference "U6") (unit 1)
+        )
+      )
+    )
+  )
+  (symbol (lib_id "Device:LED") (at 130 140 0) (unit 1)
+    (in_bom yes) (on_board yes)
+    (property "Reference" "D3" (at 130 127.3 0)
+      (effects (font (size 1.27 1.27)))
+    )
+    (property "Value" "IR neck" (at 130 152.7 0)
+      (effects (font (size 1.27 1.27)))
+    )
+    (property "Footprint" "LED_SMD:LED_0805_2012Metric" (at 130 140 0)
+      (effects (font (size 1.27 1.27)) hide)
+    )
+    (property "Datasheet" "~" (at 130 140 0)
+      (effects (font (size 1.27 1.27)) hide)
+    )
+    (pin "1")
+    (pin "2")
+    (instances
+      (project "collar-reva"
+        (path "/7fffe17a-9ffb-4f1f-b4b6-a4342b258eee/72e61ef2-c28b-4186-b83a-fe973384e252"
+          (reference "D3") (unit 1)
+        )
+      )
+    )
+  )
+  (symbol (lib_id "Device:LED") (at 155 140 0) (unit 1)
+    (in_bom yes) (on_board yes)
+    (property "Reference" "D4" (at 155 127.3 0)
+      (effects (font (size 1.27 1.27)))
+    )
+    (property "Value" "PD neck" (at 155 152.7 0)
+      (effects (font (size 1.27 1.27)))
+    )
+    (property "Footprint" "Diode_SMD:D_0805_2012Metric" (at 155 140 0)
+      (effects (font (size 1.27 1.27)) hide)
+    )
+    (property "Datasheet" "~" (at 155 140 0)
+      (effects (font (size 1.27 1.27)) hide)
+    )
+    (pin "1")
+    (pin "2")
+    (instances
+      (project "collar-reva"
+        (path "/7fffe17a-9ffb-4f1f-b4b6-a4342b258eee/72e61ef2-c28b-4186-b83a-fe973384e252"
+          (reference "D4") (unit 1)
+        )
+      )
+    )
+  )
+  (symbol (lib_id "Device:LED") (at 130 155 0) (unit 1)
+    (in_bom yes) (on_board yes)
+    (property "Reference" "D5" (at 130 142.3 0)
+      (effects (font (size 1.27 1.27)))
+    )
+    (property "Value" "RED neck" (at 130 167.7 0)
+      (effects (font (size 1.27 1.27)))
+    )
+    (property "Footprint" "LED_SMD:LED_0805_2012Metric" (at 130 155 0)
+      (effects (font (size 1.27 1.27)) hide)
+    )
+    (property "Datasheet" "~" (at 130 155 0)
+      (effects (font (size 1.27 1.27)) hide)
+    )
+    (pin "1")
+    (pin "2")
+    (instances
+      (project "collar-reva"
+        (path "/7fffe17a-9ffb-4f1f-b4b6-a4342b258eee/72e61ef2-c28b-4186-b83a-fe973384e252"
+          (reference "D5") (unit 1)
+        )
+      )
+    )
+  )
+  (symbol (lib_id "Device:R") (at 50 160 0) (unit 1)
+    (in_bom yes) (on_board yes)
+    (property "Reference" "RT1" (at 50 147.3 0)
+      (effects (font (size 1.27 1.27)))
+    )
+    (property "Value" "10k NTC" (at 50 172.7 0)
+      (effects (font (size 1.27 1.27)))
+    )
+    (property "Footprint" "Resistor_SMD:R_0402_1005Metric" (at 50 160 0)
+      (effects (font (size 1.27 1.27)) hide)
+    )
+    (property "Datasheet" "~" (at 50 160 0)
+      (effects (font (size 1.27 1.27)) hide)
+    )
+    (pin "1")
+    (pin "2")
+    (instances
+      (project "collar-reva"
+        (path "/7fffe17a-9ffb-4f1f-b4b6-a4342b258eee/72e61ef2-c28b-4186-b83a-fe973384e252"
+          (reference "RT1") (unit 1)
+        )
+      )
+    )
+  )
+  (symbol (lib_id "Device:R") (at 50 145 0) (unit 1)
+    (in_bom yes) (on_board yes)
+    (property "Reference" "R11" (at 50 132.3 0)
+      (effects (font (size 1.27 1.27)))
+    )
+    (property "Value" "10k NTC" (at 50 157.7 0)
+      (effects (font (size 1.27 1.27)))
+    )
+    (property "Footprint" "Resistor_SMD:R_0402_1005Metric" (at 50 145 0)
+      (effects (font (size 1.27 1.27)) hide)
+    )
+    (property "Datasheet" "~" (at 50 145 0)
+      (effects (font (size 1.27 1.27)) hide)
+    )
+    (pin "1")
+    (pin "2")
+    (instances
+      (project "collar-reva"
+        (path "/7fffe17a-9ffb-4f1f-b4b6-a4342b258eee/72e61ef2-c28b-4186-b83a-fe973384e252"
+          (reference "R11") (unit 1)
+        )
+      )
+    )
+  )
+  (symbol (lib_id "Device:C") (at 55 140 0) (unit 1)
+    (in_bom yes) (on_board yes)
+    (property "Reference" "C8" (at 55 127.3 0)
+      (effects (font (size 1.27 1.27)))
+    )
+    (property "Value" "0.1uF PPG" (at 55 152.7 0)
+      (effects (font (size 1.27 1.27)))
+    )
+    (property "Footprint" "Capacitor_SMD:C_0402_1005Metric" (at 55 140 0)
+      (effects (font (size 1.27 1.27)) hide)
+    )
+    (property "Datasheet" "~" (at 55 140 0)
+      (effects (font (size 1.27 1.27)) hide)
+    )
+    (pin "1")
+    (pin "2")
+    (instances
+      (project "collar-reva"
+        (path "/7fffe17a-9ffb-4f1f-b4b6-a4342b258eee/72e61ef2-c28b-4186-b83a-fe973384e252"
+          (reference "C8") (unit 1)
+        )
+      )
+    )
+  )
   (symbol (lib_id "Device:R") (at 110 45 0) (unit 1)
     (in_bom yes) (on_board yes)
@@
       (effects (font (size 1.27 1.27)))
     )
-    (property "Footprint" "" (at 110 45 0)
+    (property "Footprint" "Resistor_SMD:R_0402_1005Metric" (at 110 45 0)
       (effects (font (size 1.27 1.27)) hide)
     )
@@
       (effects (font (size 1.27 1.27)))
     )
-    (property "Footprint" "" (at 125 45 0)
+    (property "Footprint" "Resistor_SMD:R_0402_1005Metric" (at 125 45 0)
       (effects (font (size 1.27 1.27)) hide)
     )
@@
       (effects (font (size 1.27 1.27)))
     )
-    (property "Footprint" "" (at 80 95 0)
+    (property "Footprint" "Capacitor_SMD:C_0402_1005Metric" (at 80 95 0)
       (effects (font (size 1.27 1.27)) hide)
     )
@@
       (effects (font (size 1.27 1.27)))
     )
-    (property "Footprint" "" (at 160 95 0)
+    (property "Footprint" "Capacitor_SMD:C_0402_1005Metric" (at 160 95 0)
       (effects (font (size 1.27 1.27)) hide)
     )
@@
     (effects (font (size 1.27 1.27)) (justify left))
   )
+  (global_label "PPG_RDY" (shape input) (at 100 132.38 0) (fields_autoplaced)
+    (effects (font (size 1.27 1.27)) (justify left))
+  )
+  (global_label "PPG_RST" (shape input) (at 100 134.92 0) (fields_autoplaced)
+    (effects (font (size 1.27 1.27)) (justify left))
+  )
+  (global_label "PPG_TXP" (shape input) (at 145 140 0) (fields_autoplaced)
+    (effects (font (size 1.27 1.27)) (justify left))
+  )
+  (global_label "PPG_TX2" (shape input) (at 145 155 0) (fields_autoplaced)
+    (effects (font (size 1.27 1.27)) (justify left))
+  )
+  (global_label "PPG_INP" (shape input) (at 170 140 0) (fields_autoplaced)
+    (effects (font (size 1.27 1.27)) (justify left))
+  )
+  (global_label "SKIN_SENSE" (shape input) (at 55 160 0) (fields_autoplaced)
+    (effects (font (size 1.27 1.27)) (justify left))
+  )
+  (global_label "SDA" (shape input) (at 60 142.54 0) (fields_autoplaced)
+    (effects (font (size 1.27 1.27)) (justify left))
+  )
+  (global_label "SCL" (shape input) (at 60 140 0) (fields_autoplaced)
+    (effects (font (size 1.27 1.27)) (justify left))
+  )
